File: ch341-to-mfi-chip.kicad_sch (KiCad schematic)
At the start: 14 parts, among them J1 USB-212-BCW, U1 CH341F, U2 HR1117V-3.3, U3 MFI337S3959

Commit message: now better
Changed lines of the file:
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@@
+	(wire
+		(pts
+			(xy 53.34 50.8) (xy 53.34 63.5)
+		)
+		(stroke
+			(width 0)
+			(type default)
+		)
+	)
 	(wire
 		(pts
@@
 	(symbol
 		(lib_id "power:GND")
-		(at 53.34 63.5 180)
+		(at 53.34 50.8 180)
 		(unit 1)
 		(body_style 1)
@@
 		(fields_autoplaced yes)
 		(property "Reference" "#PWR09"
-			(at 53.34 57.15 0)
+			(at 53.34 44.45 0)
 			(hide yes)
 			(show_name no)
@@
 		)
 		(property "Value" "GND"
-			(at 53.34 58.42 0)
+			(at 53.34 45.72 0)
 			(show_name no)
 			(do_not_autoplace no)
@@
 		)
 		(property "Footprint" ""
-			(at 53.34 63.5 0)
+			(at 53.34 50.8 0)
 			(hide yes)
 			(show_name no)
@@
 		)
 		(property "Datasheet" ""
-			(at 53.34 63.5 0)
+			(at 53.34 50.8 0)
 			(hide yes)
 			(show_name no)
@@
 		)
 		(property "Description" "Power symbol creates a global label with name \"GND\" , ground"
-			(at 53.34 63.5 0)
-			(hide yes)
-			(show_name no)
+			(at 53.34 50.8 0)
+			(hide yes)
+			(show_name no)
