File: USBA-5V-CH341-MFI337S3959/ch341-to-mfi-chip.kicad_sch (KiCad schematic)
At the start: 13 parts, among them J1 USB-212-BCW, U1 CH341F, U2 HR1117V-3.3, U3 MFI337S3959

Commit message: add tiny layout of the dongle
Parts:
- removed C2: 10uF, Capacitor_SMD:C_0402_1005Metric, symbol Device:C
- removed U2: HR1117V-3.3, Package_TO_SOT_SMD:SOT-89-3, symbol Regulator_Linear:LT1083-3.3
Connections:
- net +3V3 is gone; now on net +5V: C1.1, C3.1, C4.1, C5.2, R2.1, R3.1, R4.1, U1.28 (VCC), U1.9 (V3), U3.8 (VCC)
- net +5V: now reaches J1.1 (VBUS)
