File: dev-USBA-3.3V-CH341-MFI337S3959/ch341-to-mfi-chip.kicad_sch (KiCad schematic)
At the start: 13 parts, among them J1 USB-212-BCW, U1 CH341F, U2 HR1117V-3.3, U3 MFI337S3959

Commit message: add tiny layout of the dongle
Parts:
- added R5: 4.7k, Resistor_SMD:R_0402_1005Metric, symbol Device:R
- J1: footprint footprint:917-511A1015B20200 -> Connector_USB:USB_A_Connfly_DS1098_Horizontal
Connections:
- net GND: now also R5.2
- net at R4.2, U1.15 (CS0), U3.7 (RST): now also R5.1
Changed lines of the file:
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@@
+	)
+	(junction
+		(at 83.82 73.66)
+		(diameter 0)
+		(color 0 0 0 0)
 	)
 	(junction
@@
 	(wire
 		(pts
-			(xy 82.55 73.66) (xy 91.44 73.66)
+			(xy 82.55 73.66) (xy 83.82 73.66)
 		)
 		(stroke
@@
 	(wire
 		(pts
+			(xy 83.82 91.44) (xy 92.71 91.44)
+		)
+		(stroke
+			(width 0)
+			(type default)
+		)
+	)
+	(wire
+		(pts
 			(xy 93.98 39.37) (xy 101.6 39.37)
 		)
@@
 	(wire
 		(pts
+			(xy 83.82 73.66) (xy 83.82 76.2)
+		)
+		(stroke
+			(width 0)
+			(type default)
+		)
+	)
+	(wire
+		(pts
 			(xy 189.23 46.99) (xy 189.23 48.26)
 		)
@@
 	(wire
 		(pts
+			(xy 83.82 73.66) (xy 91.44 73.66)
+		)
+		(stroke
+			(width 0)
+			(type default)
+		)
+	)
+	(wire
+		(pts
 			(xy 105.41 78.74) (xy 105.41 93.98)
 		)
@@
 		(pts
 			(xy 101.6 39.37) (xy 101.6 45.72)
+		)
+		(stroke
+			(width 0)
+			(type default)
+		)
+	)
+	(wire
+		(pts
+			(xy 83.82 83.82) (xy 83.82 91.44)
 		)
 		(stroke
@@
 	)
 	(symbol
+		(lib_id "Device:R")
+		(at 83.82 80.01 0)
+		(unit 1)
+		(body_style 1)
+		(exclude_from_sim no)
+		(in_bom yes)
+		(on_board yes)
+		(in_pos_files yes)
+		(dnp yes)
+		(fields_autoplaced yes)
+		(property "Reference" "R5"
+			(at 86.36 78.7399 0)
+			(show_name no)
+			(do_not_autoplace no)
+			(effects
+				(font
+					(size 1.27 1.27)
+				)
+				(justify left)
+			)
+		)
+		(property "Value" "4.7k"
+			(at 86.36 81.2799 0)
+			(show_name no)
+			(do_not_autoplace no)
+			(effects
+				(font
+					(size 1.27 1.27)
+				)
+				(justify left)
+			)
+		)
+		(property "Footprint" "Resistor_SMD:R_0402_1005Metric"
+			(at 82.042 80.01 90)
+			(hide yes)
+			(show_name no)
+			(do_not_autoplace no)
+			(effects
+				(font
+					(size 1.27 1.27)
+				)
+			)
+		)
+		(property "Datasheet" ""
+			(at 83.82 80.01 0)
+			(hide yes)
+			(show_name no)
+			(do_not_autoplace no)
+			(effects
+				(font
+					(size 1.27 1.27)
+				)
+			)
+		)
+		(property "Description" "Resistor"
+			(at 83.82 80.01 0)
+			(hide yes)
+			(show_name no)
+			(do_not_autoplace no)
+			(effects
+				(font
+					(size 1.27 1.27)
+				)
+			)
+		)
+		(pin "2"
+		)
+		(pin "1"
+		)
+		(instances
+			(project "ch341-to-mfi-chip"
+				(path "/5362e1ec-2bd0-4b31-b6ed-5b973739ecf7"
+					(reference "R5")
+					(unit 1)
+				)
+			)
+		)
+	)
+	(symbol
 		(lib_id "Connector:USB_A")
 		(at 162.56 71.12 0)
@@
 			)
 		)
-		(property "Footprint" "footprint:917-511A1015B20200"
+		(property "Footprint" "Connector_USB:USB_A_Connfly_DS1098_Horizontal"
 			(at 158.75 72.39 0)
 			(hide yes)
